File: hardware/src/cansat_pcb.kicad_pcb (KiCad board)
At the start: 2 copper layers, 7 parts, among them J1 Servo_motor, J2 Sen057_pressure_sensor, J3 Hall_effect_sensor, J4 Jack plug, SW1 SPDT_Slide_SMD_6.7x2.6mm, U1 XIAO-nRF52840-Plus-SMD

Commit message: feature: add some componants to the pcb
Parts:
- removed J4: Jack plug, Connector_PinHeader_1.00mm:PinHeader_1x02_P1.00mm_Horizontal
- added Btn: telemetry_btn, craby's_library:SW_BUTT-2, B.Cu at (120.1, 99.0)
- added Jack: Jack plug, Connector_PinHeader_2.54mm:PinHeader_1x02_P2.54mm_Horizontal, B.Cu at (110.0, 97.4)
- Mcu: renamed from U1; moved to B.Cu
- Sw: renamed from SW1; moved to B.Cu
- moved Motor 40.1 mm to (148.7, 85.4)
- moved BME 28.9 mm to (142.9, 80.5)
- moved Pressure 28.8 mm to (142.9, 90.4)
- moved Sw 5.54 mm to (134.7, 85.3), turned to -90 degrees
- moved Bz 3.57 mm to (128.4, 101.7)
- turned Mcu to 180 degrees
- renumbered J3 to BME, BZ1 to Bz, J1 to Motor, J2 to Pressure
